File: Hardware/testhologram v2/testhologram v2/testhologram v2.kicad_sch (KiCad schematic)
At the start: 696 parts, among them J1 USB_C_Receptacle_USB2.0_16P, J2 Conn_01x06_Socket, SW1 SW_Reset, SW2 SW_Boot, SW3 SW_opt1, SW4 SW_opt2, U1 SM16106SC, U10 SM16106SC, U11 SM16106SC, U12 SM16106SC, U13 SM16106SC, U14 SM16106SC, U15 SM16106SC, U16 SM16106SC, U17 SM16106SC, U18 SM16106SC, U19 SM16106SC, U2 SM16106SC, U20 SM16106SC, U21 SM16106SC, U22 SM16106SC, U23 SM16106SC, U24 SM16106SC, U25 SM16106SC, U26 SM16106SC, U27 SM16106SC, U28 SM16106SC, U29 SM16106SC, U3 SM16106SC, U30 SM16106SC, U31 SM16106SC, U32 SM16106SC, U33 ESP32-S3-WROOM-1(N16R8), U34 SY8286ARAC 12v->4v, U36 SY8286ARAC 12v->3.3v, U4 SM16106SC, U5 SM16106SC, U6 SM16106SC, U7 SM16106SC, U8 SM16106SC, U9 SM16106SC

Commit message: finished schematic, working on pcb design
Parts:
- added H1: topLeft, MountingHole:MountingHole_5mm_Pad, symbol Mechanical:MountingHole
- added H2: topRight, MountingHole:MountingHole_5mm_Pad, symbol Mechanical:MountingHole
- added H3: botLeft, MountingHole:MountingHole_5mm_Pad, symbol Mechanical:MountingHole
- added H4: botRight, MountingHole:MountingHole_5mm_Pad, symbol Mechanical:MountingHole
- J2: footprint (none) -> TerminalBlock:TerminalBlock_MaiXu_MX126-5.0-06P_1x06_P5.00mm; symbol Connector:Conn_01x06_Socket -> Connector:Screw_Terminal_01x06
- R33, R34, R35, R36, R37, R38, R39, R40, R41, R47, R48, R51, R52, R53, R54, R56, R57, R58, R59, R60, R61, R62, R63, R64: footprint (none) -> Resistor_SMD:R_0603_1608Metric
- R42, R43, R44, R45, R46, R49, R50, R55, R65, R66: footprint (none) -> Resistor_SMD:R_0402_1005Metric
- SW1, SW2: footprint (none) -> easyeda:KEY-SMD_L4.0-W3.0-LS4.9-1
- U1, U10, U11, U12, U13, U14, U15, U16, U17, U18, U19, U2, U20, U21, U22, U23, U24, U25, U26, U27, U28, U29, U3, U30, U31, U32, U4, U5, U6, U7, U8, U9: footprint easyeda2kicad:QSOP-24_L8.7-W4.0-P0.65-LS6.0-BL -> easyeda:QSOP-24_L8.7-W4.0-P0.64-LS6.0-BL
- U33: footprint easyeda2kicad:WIRELM-SMD_ESP32-S3-WROOM-1 -> easyeda:WIRELM-SMD_ESP32-S3-WROOM-1
